File: Power.kicad_sch (KiCad schematic)
At the start: 11 parts, among them U2 AMS1117-3.3

Commit message: switch caps for lower cost
Parts:
- C3, C5: P/N C0603G104K5RACT250 -> UMK107B7104KAHT
Changed lines of the file:
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@@
 			)
 		)
-		(property "P/N" "C0603G104K5RACT250"
+		(property "P/N" "UMK107B7104KAHT "
 			(at 106.68 38.1 0)
 			(effects
@@
 			)
 		)
-		(property "P/N" "C0603G104K5RACT250"
+		(property "P/N" "UMK107B7104KAHT "
 			(at 83.82 38.1 0)
 			(effects
