File: Switches.kicad_sch (KiCad schematic)
At the start: 6 parts, among them SW1 BOOT, SW2 RST

Commit message: finished sch? (need P/Ns)
Parts:
- added C11, C12: 0.1u, symbol Device:C
- added R8, R9: 10k, symbol Device:R
- added SW3: FLIP, symbol Switch:SW_Push
- added SW4: FLOP, symbol Switch:SW_Push
Connections:
- net +3.3V: now also R8.1, R9.1
- net GND: now also C11.2, C12.2, SW3.1, SW4.1
- new net FLIP: C11.1, R8.2, SW3.2
- new net FLOP: C12.1, R9.2, SW4.2

Commit message: add P/N
Parts:
- C11, C12, C6, C7: P/N (none) -> C0603G104K5RACT250
- R4, R5, R8, R9: P/N (none) -> MCT0603PD1002DP500
- SW1, SW2, SW3, SW4: P/N (none) -> TL6120AF160QG
Changed lines of the file:
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@@
+			)
+		)
+		(property "P/N" "C0603G104K5RACT250"
+			(at 38.1 41.91 0)
+			(effects
+				(font
+					(size 1.27 1.27)
+				)
+				(hide yes)
 			)
 		)
@@
 			)
 		)
+		(property "P/N" "MCT0603PD1002DP500"
+			(at 38.1 29.21 0)
+			(effects
+				(font
+					(size 1.27 1.27)
+				)
+				(hide yes)
+			)
+		)
 		(pin "2"
 		)
@@
 			)
 		)
+		(property "P/N" "MCT0603PD1002DP500 "
+			(at 115.57 29.21 0)
+			(effects
+				(font
+					(size 1.27 1.27)
+				)
+				(hide yes)
+			)
+		)
 		(pin "2"
 		)
@@
 			)
 		)
+		(property "P/N" "C0603G104K5RACT250"
+			(at 154.94 41.91 0)
+			(effects
+				(font
+					(size 1.27 1.27)
+				)
+				(hide yes)
+			)
+		)
 		(pin "1"
 		)
@@
 			)
 		)
+		(property "P/N" "TL6120AF160QG"
+			(at 107.95 35.56 0)
+			(effects
+				(font
+					(size 1.27 1.27)
+				)
+				(hide yes)
+			)
+		)
 		(pin "2"
 		)
@@
 			)
 		)
+		(property "P/N" "TL6120AF160QG"
+			(at 147.32 35.56 0)
+			(effects
+				(font
+					(size 1.27 1.27)
+				)
+				(hide yes)
+			)
+		)
 		(pin "2"
 		)
@@
 			)
 		)
+		(property "P/N" "TL6120AF160QG"
+			(at 30.48 35.56 0)
+			(effects
+				(font
+					(size 1.27 1.27)
+				)
+				(hide yes)
+			)
+		)
 		(pin "2"
 		)
@@
 			)
 		)
+		(property "P/N" "MCT0603PD1002DP500"
+			(at 77.47 29.21 0)
+			(effects
+				(font
+					(size 1.27 1.27)
+				)
+				(hide yes)
+			)
+		)
 		(pin "2"
 		)
@@
 			)
 		)
+		(property "P/N" "MCT0603PD1002DP500"
+			(at 154.94 29.21 0)
+			(effects
+				(font
+					(size 1.27 1.27)
+				)
+				(hide yes)
+			)
+		)
 		(pin "2"
 		)
@@
 			)
 		)
+		(property "P/N" "C0603G104K5RACT250"
+			(at 77.47 41.91 0)
+			(effects
+				(font
+					(size 1.27 1.27)
+				)
+				(hide yes)
+			)
+		)
 		(pin "1"
 		)
@@
 			)
 		)
+		(property "P/N" "TL6120AF160QG"
+			(at 69.85 35.56 0)
+			(effects
+				(font
+					(size 1.27 1.27)
+				)
+				(hide yes)
+			)
+		)
 		(pin "2"
 		)
@@
 			(at 115.57 41.91 0)
 			(effects
+				(font
+					(size 1.27 1.27)
+				)
+				(hide yes)
+			)
+		)
+		(property "P/N" "C0603G104K5RACT250"
+			(at 115.57 41.91 0)
+			(effects

Commit message: assign footprints
Parts:
- C11, C12, C6, C7: footprint (none) -> Capacitor_SMD:C_0603_1608Metric
- R4, R5, R8, R9: footprint (none) -> Resistor_SMD:R_0603_1608Metric
- SW1, SW2, SW3, SW4: footprint (none) -> Button_Switch_SMD:SW_Push_1P1T_NO_CK_KMR2; P/N TL6120AF160QG -> KMR231GLFS
Changed lines of the file:
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@@
 			)
 		)
-		(property "Footprint" ""
+		(property "Footprint" "Capacitor_SMD:C_0603_1608Metric"
 			(at 39.0652 45.72 0)
 			(effects
@@
 			)
 		)
-		(property "Footprint" ""
+		(property "Footprint" "Resistor_SMD:R_0603_1608Metric"
 			(at 36.322 29.21 90)
 			(effects
@@
 			)
 		)
-		(property "Footprint" ""
+		(property "Footprint" "Resistor_SMD:R_0603_1608Metric"
 			(at 113.792 29.21 90)
 			(effects
@@
 			)
 		)
-		(property "Footprint" ""
+		(property "Footprint" "Capacitor_SMD:C_0603_1608Metric"
 			(at 155.9052 45.72 0)
 			(effects
@@
 			)
 		)
-		(property "Footprint" ""
+		(property "Footprint" "Button_Switch_SMD:SW_Push_1P1T_NO_CK_KMR2"
 			(at 107.95 30.48 0)
 			(effects
@@
 			)
 		)
-		(property "P/N" "TL6120AF160QG"
+		(property "P/N" "KMR231GLFS"
 			(at 107.95 35.56 0)
 			(effects
@@
 			)
 		)
-		(property "Footprint" ""
+		(property "Footprint" "Button_Switch_SMD:SW_Push_1P1T_NO_CK_KMR2"
 			(at 147.32 30.48 0)
 			(effects
@@
 			)
 		)
-		(property "P/N" "TL6120AF160QG"
+		(property "P/N" "KMR231GLFS"
 			(at 147.32 35.56 0)
 			(effects
@@
 			)
 		)
-		(property "Footprint" ""
+		(property "Footprint" "Button_Switch_SMD:SW_Push_1P1T_NO_CK_KMR2"
 			(at 30.48 30.48 0)
 			(effects
@@
 			)
 		)
-		(property "P/N" "TL6120AF160QG"
+		(property "P/N" "KMR231GLFS"
 			(at 30.48 35.56 0)
 			(effects
@@
 			)
 		)
-		(property "Footprint" ""
+		(property "Footprint" "Resistor_SMD:R_0603_1608Metric"
 			(at 75.692 29.21 90)
 			(effects
@@
 			)
 		)
-		(property "Footprint" ""
+		(property "Footprint" "Resistor_SMD:R_0603_1608Metric"
 			(at 153.162 29.21 90)
 			(effects
@@
 			)
 		)
-		(property "Footprint" ""
+		(property "Footprint" "Capacitor_SMD:C_0603_1608Metric"
 			(at 78.4352 45.72 0)
 			(effects
@@
 			)
 		)
-		(property "Footprint" ""
+		(property "Footprint" "Button_Switch_SMD:SW_Push_1P1T_NO_CK_KMR2"
 			(at 69.85 30.48 0)
 			(effects
@@
 			)
 		)
-		(property "P/N" "TL6120AF160QG"
+		(property "P/N" "KMR231GLFS"
 			(at 69.85 35.56 0)
 			(effects
@@
 			)
 		)
-		(property "Footprint" ""
+		(property "Footprint" "Capacitor_SMD:C_0603_1608Metric"
 			(at 116.5352 45.72 0)
 			(effects

Commit message: switch caps for lower cost
Parts:
- C11, C12, C6, C7: P/N C0603G104K5RACT250 -> UMK107B7104KAHT
Changed lines of the file:
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@@
 			)
 		)
-		(property "P/N" "C0603G104K5RACT250"
+		(property "P/N" "UMK107B7104KAHT "
 			(at 38.1 41.91 0)
 			(effects
@@
 			)
 		)
-		(property "P/N" "C0603G104K5RACT250"
+		(property "P/N" "UMK107B7104KAHT "
 			(at 154.94 41.91 0)
 			(effects
@@
 			)
 		)
-		(property "P/N" "C0603G104K5RACT250"
+		(property "P/N" "UMK107B7104KAHT "
 			(at 77.47 41.91 0)
 			(effects
@@
 			)
 		)
-		(property "P/N" "C0603G104K5RACT250"
+		(property "P/N" "UMK107B7104KAHT "
 			(at 115.57 41.91 0)
 			(effects
